File: pcb/deck module/deck module.kicad_pcb (KiCad board)
At the start: 2 copper layers, 131.5 x 167.5 mm, 51 parts, among them J1 Conn_01x04_Pin, SW1 SW_Push, SW10 SW_Push, SW11 SW_Push, SW12 SW_Push, SW13 SW_Push, SW14 SW_Push, SW15 SW_Push, SW16 SW_Push, SW17 RotaryEncoder_Switch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

Commit message: add cad
Parts:
- moved SW20 0.55 mm to (137.5, 87.5)
Routing:
- net 2a: track 90.7 -> 91.2 mm
- net 2b: track 94.3 -> 94.8 mm
